Commit message: milk calibration

File: fmauch_universal_robot/ur_description/urdf/inc/ur3_macro.xacro (robot description, xacro)
@@ -20,5 +20,5 @@
    prefix
    joint_limits_parameters_file:='$(find ur_description)/config/ur3/joint_limits.yaml'
-   kinematics_parameters_file:='$(find ur_description)/config/ur3/default_kinematics.yaml'
+   kinematics_parameters_file:='$(find ur_description)/config/ur3/milk_kinematics.yaml'
    physical_parameters_file:='$(find ur_description)/config/ur3/physical_parameters.yaml'
    visual_parameters_file:='$(find ur_description)/config/ur3/visual_parameters.yaml'

File: fmauch_universal_robot/ur_description/urdf/inc/ur_macro.xacro (robot description, xacro)
@@ -215,5 +215,5 @@
            link/frame) to introduce the necessary rotation over Z (of pi rad).
       -->
-      <origin xyz="0 0 0" rpy="0 0 ${pi}" />
+      <origin xyz="0 0 0" rpy="0 0 0" />
     </joint>
     <joint name="${prefix}shoulder_pan_joint" type="revolute">
@@ -297,5 +297,5 @@
            the UR controller.
       -->
-      <origin xyz="0 0 0" rpy="0 0 ${pi}"/>
+      <origin xyz="0 0 0" rpy="0 0 0"/>
       <parent link="${prefix}base_link"/>
       <child link="${prefix}base"/>
